File: sensor_ble/sensor_ble.sch (KiCad schematic (older format))
At the start: 23 parts, among them U1 Nrf52810-QCAA, U2 BME280, Y1 32,768KHz, Y2 32MHz

Commit message: Projeto roteado, falta a antena
Signed-off-by: Rodrigo Peixoto <rodrigopex@ic.ufal.br>
Parts:
- added FID1, FID2: Fiducial, Fiducial:Fiducial_0.5mm_Mask1.5mm, symbol Mechanical:Fiducial
- added H1, H2: MountingHole, MountingHole:MountingHole_2mm, symbol Mechanical:MountingHole
- added R3: 1k, Resistor_SMD:R_0402_1005Metric, symbol Device:R_Small_US
- BT1: footprint (none) -> Battery:Battery_Panasonic_CR2032-VS1N_Vertical_CircularHoles
- C1, C10, C11, C12, C13, C14, C2, C3, C4, C5, C6, C7, C8, C9: footprint (none) -> Capacitor_SMD:C_0402_1005Metric
- L1: footprint (none) -> Inductor_SMD:L_0402_1005Metric
- L2: footprint (none) -> Inductor_SMD:L_0805_2012Metric
- R1, R2: footprint (none) -> Resistor_SMD:R_0402_1005Metric
- U1: footprint (none) -> Package_DFN_QFN:QFN-32-1EP_5x5mm_P0.5mm_EP3.6x3.6mm
- Y1: footprint (none) -> Crystal:Crystal_SMD_3215-2Pin_3.2x1.5mm
- Y2: footprint (none) -> Crystal:Crystal_SMD_2016-4Pin_2.0x1.6mm
Connections:
- net GND: now also U1.33 (PAD), R3.2; no longer U2.5 (SDO)
- new net: R3.1, U2.5 (SDO)
- no-connect marks 17 -> 16
Changed lines of the file:
@@
 EESchema Schematic File Version 4
+LIBS:sensor_ble-cache
 EELAYER 30 0
 EELAYER END
@@
 F 0 "U1" H 3800 4550 50  0000 L CNN
 F 1 "Nrf52810-QCAA" H 3800 4450 50  0000 L CNN
-F 2 "" H 3600 5200 50  0001 C CNN
+F 2 "Package_DFN_QFN:QFN-32-1EP_5x5mm_P0.5mm_EP3.6x3.6mm" H 3600 5200 50  0001 C CNN
 F 3 "" H 3600 5200 50  0001 C CNN
 	1    4050 4450
@@
 F 0 "Y2" V 6100 3650 50  0000 L CNN
 F 1 "32MHz" V 6200 3650 50  0000 L CNN
-F 2 "" H 6100 3450 50  0001 C CNN
+F 2 "Crystal:Crystal_SMD_2016-4Pin_2.0x1.6mm" H 6100 3450 50  0001 C CNN
 F 3 "~" H 6100 3450 50  0001 C CNN
 	1    6100 3450
@@
 F 0 "C10" V 6350 3850 50  0000 C CNN
 F 1 "12pF" V 6550 3850 50  0000 C CNN
-F 2 "" H 6450 3850 50  0001 C CNN
+F 2 "Capacitor_SMD:C_0402_1005Metric" H 6450 3850 50  0001 C CNN
 F 3 "~" H 6450 3850 50  0001 C CNN
 	1    6450 3850
@@
 F 0 "C11" V 6350 4350 50  0000 C CNN
 F 1 "100pF" V 6550 4350 50  0000 C CNN
-F 2 "" H 6450 4350 50  0001 C CNN
+F 2 "Capacitor_SMD:C_0402_1005Metric" H 6450 4350 50  0001 C CNN
 F 3 "~" H 6450 4350 50  0001 C CNN
 	1    6450 4350
@@
 F 0 "C12" V 6350 4700 50  0000 C CNN
 F 1 "NF" V 6550 4700 50  0000 C CNN
-F 2 "" H 6450 4700 50  0001 C CNN
+F 2 "Capacitor_SMD:C_0402_1005Metric" H 6450 4700 50  0001 C CNN
 F 3 "~" H 6450 4700 50  0001 C CNN
 	1    6450 4700
@@
 F 0 "C8" H 4842 3246 50  0000 L CNN
 F 1 "100nF" H 4842 3155 50  0000 L CNN
-F 2 "" H 4750 3200 50  0001 C CNN
+F 2 "Capacitor_SMD:C_0402_1005Metric" H 4750 3200 50  0001 C CNN
 F 3 "~" H 4750 3200 50  0001 C CNN
 	1    4750 3200
@@
 F 0 "C5" H 3492 5846 50  0000 L CNN
 F 1 "100nF" H 3492 5755 50  0000 L CNN
-F 2 "" H 3400 5800 50  0001 C CNN
+F 2 "Capacitor_SMD:C_0402_1005Metric" H 3400 5800 50  0001 C CNN
 F 3 "~" H 3400 5800 50  0001 C CNN
 	1    3400 5800
@@
 F 0 "C4" H 3442 3196 50  0000 L CNN
 F 1 "4.7uF" H 3442 3105 50  0000 L CNN
-F 2 "" H 3350 3150 50  0001 C CNN
+F 2 "Capacitor_SMD:C_0402_1005Metric" H 3350 3150 50  0001 C CNN
 F 3 "~" H 3350 3150 50  0001 C CNN
 	1    3350 3150
@@
 F 0 "C2" V 1400 4150 50  0000 C CNN
 F 1 "12pF" V 1600 4150 50  0000 C CNN
-F 2 "" H 1500 4150 50  0001 C CNN
+F 2 "Capacitor_SMD:C_0402_1005Metric" H 1500 4150 50  0001 C CNN
 F 3 "~" H 1500 4150 50  0001 C CNN
 	1    1500 4150
@@
 F 0 "C1" V 1400 3600 50  0000 C CNN
 F 1 "12pF" V 1600 3600 50  0000 C CNN
-F 2 "" H 1500 3600 50  0001 C CNN
+F 2 "Capacitor_SMD:C_0402_1005Metric" H 1500 3600 50  0001 C CNN
 F 3 "~" H 1500 3600 50  0001 C CNN
 	1    1500 3600
@@
 F 0 "Y1" V 1854 4031 50  0000 L CNN
 F 1 "32,768KHz" V 1945 4031 50  0000 L CNN
-F 2 "" H 1900 3900 50  0001 C CNN
+F 2 "Crystal:Crystal_SMD_3215-2Pin_3.2x1.5mm" H 1900 3900 50  0001 C CNN
 F 3 "~" H 1900 3900 50  0001 C CNN
 	1    1900 3900
@@
 F 0 "C3" H 2742 3796 50  0000 L CNN
 F 1 "100nF" H 2742 3705 50  0000 L CNN
-F 2 "" H 2650 3750 50  0001 C CNN
+F 2 "Capacitor_SMD:C_0402_1005Metric" H 2650 3750 50  0001 C CNN
 F 3 "~" H 2650 3750 50  0001 C CNN
 	1    2650 3750
@@
 F 0 "C6" H 4342 2346 50  0000 L CNN
 F 1 "1uF" H 4342 2255 50  0000 L CNN
-F 2 "" H 4250 2300 50  0001 C CNN
+F 2 "Capacitor_SMD:C_0402_1005Metric" H 4250 2300 50  0001 C CNN
 F 3 "~" H 4250 2300 50  0001 C CNN
 	1    4250 2300
@@
 F 0 "C7" H 4792 2346 50  0000 L CNN
 F 1 "N.F." H 4792 2255 50  0000 L CNN
-F 2 "" H 4700 2300 50  0001 C CNN
+F 2 "Capacitor_SMD:C_0402_1005Metric" H 4700 2300 50  0001 C CNN
 F 3 "~" H 4700 2300 50  0001 C CNN
 	1    4700 2300
@@
 F 0 "L2" H 3653 2696 50  0000 L CNN
 F 1 "10uH" H 3653 2605 50  0000 L CNN
-F 2 "" H 3600 2650 50  0001 C CNN
+F 2 "Inductor_SMD:L_0805_2012Metric" H 3600 2650 50  0001 C CNN
 F 3 "~" H 3600 2650 50  0001 C CNN
 	1    3600 2650
@@
 F 0 "L1" H 3653 2396 50  0000 L CNN
 F 1 "15nH" H 3653 2305 50  0000 L CNN
-F 2 "" H 3600 2350 50  0001 C CNN
+F 2 "Inductor_SMD:L_0402_1005Metric" H 3600 2350 50  0001 C CNN
 F 3 "~" H 3600 2350 50  0001 C CNN
 	1    3600 2350
@@
 F 0 "C9" V 6350 3250 50  0000 C CNN
 F 1 "12pF" V 6550 3250 50  0000 C CNN
-F 2 "" H 6450 3250 50  0001 C CNN
+F 2 "Capacitor_SMD:C_0402_1005Metric" H 6450 3250 50  0001 C CNN
 F 3 "~" H 6450 3250 50  0001 C CNN
 	1    6450 3250
@@
 F 0 "C13" H 9042 2096 50  0000 L CNN
 F 1 "100nF" H 9042 2005 50  0000 L CNN
-F 2 "" H 8950 2050 50  0001 C CNN
+F 2 "Capacitor_SMD:C_0402_1005Metric" H 8950 2050 50  0001 C CNN
 F 3 "~" H 8950 2050 50  0001 C CNN
 	1    8950 2050
@@
 F 0 "C14" H 10092 2096 50  0000 L CNN
 F 1 "100nF" H 10092 2005 50  0000 L CNN
-F 2 "" H 10000 2050 50  0001 C CNN
+F 2 "Capacitor_SMD:C_0402_1005Metric" H 10000 2050 50  0001 C CNN
 F 3 "~" H 10000 2050 50  0001 C CNN
 	1    10000 2050
@@
 Wire Wire Line
 	10050 3200 10400 3200
-$Comp
-L power:GND #PWR023
-U 1 1 5DD2544B
-P 10400 2650
-F 0 "#PWR023" H 10400 2400 50  0001 C CNN
-F 1 "GND" H 10405 2477 50  0000 C CNN
-F 2 "" H 10400 2650 50  0001 C CNN
-F 3 "" H 10400 2650 50  0001 C CNN
-	1    10400 2650
-	1    0    0    -1
-$EndComp
-Wire Wire Line
-	10050 2600 10400 2600
-Wire Wire Line
-	10400 2600 10400 2650
 Wire Wire Line
 	10050 3000 10100 3000
@@
 F 0 "R1" H 2218 4596 50  0000 L CNN
 F 1 "4,7k" H 2218 4505 50  0000 L CNN
-F 2 "" H 2150 4550 50  0001 C CNN
+F 2 "Resistor_SMD:R_0402_1005Metric" H 2150 4550 50  0001 C CNN
 F 3 "~" H 2150 4550 50  0001 C CNN
 	1    2150 4550
@@
 F 0 "R2" H 2568 4596 50  0000 L CNN
 F 1 "4,7k" H 2568 4505 50  0000 L CNN
-F 2 "" H 2500 4550 50  0001 C CNN
+F 2 "Resistor_SMD:R_0402_1005Metric" H 2500 4550 50  0001 C CNN
 F 3 "~" H 2500 4550 50  0001 C CNN
 	1    2500 4550
@@
 F 0 "BT1" H 9568 5696 50  0000 L CNN
 F 1 "Battery_Cell" H 9568 5605 50  0000 L CNN
-F 2 "" V 9450 5660 50  0001 C CNN
+F 2 "Battery:Battery_Panasonic_CR2032-VS1N_Vertical_CircularHoles" V 9450 5660 50  0001 C CNN
 F 3 "~" V 9450 5660 50  0001 C CNN
 	1    9450 5600
@@
 NoConn ~ 4300 3450
 NoConn ~ 5050 4450
-NoConn ~ 5050 4550
 NoConn ~ 5050 4650
 NoConn ~ 5050 4750
@@
 	1    0    0    -1
 $EndComp
+$Comp
+L power:GND #PWR023
+U 1 1 5DD2544B
+P 10650 2850
+F 0 "#PWR023" H 10650 2600 50  0001 C CNN
+F 1 "GND" H 10655 2677 50  0000 C CNN
+F 2 "" H 10650 2850 50  0001 C CNN
+F 3 "" H 10650 2850 50  0001 C CNN
+	1    10650 2850
+	1    0    0    -1
+$EndComp
+$Comp
+L Device:R_Small_US R3
+U 1 1 5DD8A3B2
+P 10650 2750
+F 0 "R3" H 10718 2796 50  0000 L CNN
+F 1 "1k" H 10718 2705 50  0000 L CNN
+F 2 "Resistor_SMD:R_0402_1005Metric" H 10650 2750 50  0001 C CNN
+F 3 "~" H 10650 2750 50  0001 C CNN
+	1    10650 2750
+	1    0    0    -1
+$EndComp
+Wire Wire Line
+	10050 2600 10650 2600
+Wire Wire Line
+	10650 2600 10650 2650
+Wire Wire Line
+	3600 3450 3600 3250
+Wire Wire Line
+	3600 3250 3350 3250
+Connection ~ 3350 3250
+$Comp
+L Mechanical:Fiducial FID1
+U 1 1 5DE2F9CF
+P 2150 7150
+F 0 "FID1" H 2235 7196 50  0000 L CNN
+F 1 "Fiducial" H 2235 7105 50  0000 L CNN
+F 2 "Fiducial:Fiducial_0.5mm_Mask1.5mm" H 2150 7150 50  0001 C CNN
+F 3 "~" H 2150 7150 50  0001 C CNN
+	1    2150 7150
+	1    0    0    -1
+$EndComp
+$Comp
+L Mechanical:Fiducial FID2
+U 1 1 5DE312B7
+P 2850 7150
+F 0 "FID2" H 2935 7196 50  0000 L CNN
+F 1 "Fiducial" H 2935 7105 50  0000 L CNN
+F 2 "Fiducial:Fiducial_0.5mm_Mask1.5mm" H 2850 7150 50  0001 C CNN
+F 3 "~" H 2850 7150 50  0001 C CNN
+	1    2850 7150
+	1    0    0    -1
+$EndComp
+$Comp
+L Mechanical:MountingHole H1
+U 1 1 5DE3894B
+P 3650 7150
+F 0 "H1" H 3750 7196 50  0000 L CNN
+F 1 "MountingHole" H 3750 7105 50  0000 L CNN
+F 2 "MountingHole:MountingHole_2mm" H 3650 7150 50  0001 C CNN
+F 3 "~" H 3650 7150 50  0001 C CNN
+	1    3650 7150
+	1    0    0    -1
+$EndComp
+$Comp
+L Mechanical:MountingHole H2
+U 1 1 5DE39090
+P 4300 7150
+F 0 "H2" H 4400 7196 50  0000 L CNN
+F 1 "MountingHole" H 4400 7105 50  0000 L CNN
+F 2 "MountingHole:MountingHole_2mm" H 4300 7150 50  0001 C CNN
+F 3 "~" H 4300 7150 50  0001 C CNN
+	1    4300 7150
+	1    0    0    -1
+$EndComp

Commit message: Adiciona antena
Signed-off-by: Rodrigo Peixoto <rodrigopex@ic.ufal.br>
Parts:
- added AE1: Antenna_Chip, sensor_ble:2450AT18B100, symbol Device:Antenna_Chip
- added J1: TC2030, Connector:Tag-Connect_TC2030-IDC-NL_2x03_P1.27mm_Vertical, symbol Connector_Generic:Conn_02x03_Odd_Even
- added R4, R6: NC, Resistor_SMD:R_0402_1005Metric, symbol Device:R_Small_US
- added R5: 0, Resistor_SMD:R_0402_1005Metric, symbol Device:R_Small_US
Connections:
- net GND: now also J1.5 (Pin_5), R4.1
- net VDD: now also J1.1 (Pin_1)
- net NRESET: now reaches U1.16 (P0.21/RESET)
- net NRESET: now also J1.3 (Pin_3)
- net SWCLK: now reaches U1.17 (SWDCLK)
- net SWCLK: now also J1.4 (Pin_4)
- net SWDIO: now reaches U1.18 (SWDIO)
- net SWDIO: now also J1.2 (Pin_2)
- net ANT: now reaches U1.19 (ANT)
- net ANT: now also R6.2
- new net: AE1.1 (FEED), R5.1
- new net: R4.2, R5.2, R6.1
- no-connect marks 16 -> 15
Changed lines of the file:
@@
 $EndDescr
-$Comp
-L sensor_ble:Nrf52810-QCAA U1
-U 1 1 5DC5E292
-P 4050 4450
-F 0 "U1" H 3800 4550 50  0000 L CNN
-F 1 "Nrf52810-QCAA" H 3800 4450 50  0000 L CNN
-F 2 "Package_DFN_QFN:QFN-32-1EP_5x5mm_P0.5mm_EP3.6x3.6mm" H 3600 5200 50  0001 C CNN
-F 3 "" H 3600 5200 50  0001 C CNN
-	1    4050 4450
-	1    0    0    -1
-$EndComp
 $Comp
 L power:GND #PWR013
@@
 NoConn ~ 4300 3450
 NoConn ~ 5050 4450
-NoConn ~ 5050 4650
-NoConn ~ 5050 4750
 NoConn ~ 3100 4400
 NoConn ~ 3100 4500
@@
 NoConn ~ 4200 5400
 NoConn ~ 4300 5400
-NoConn ~ 4400 5400
 $Comp
 L power:PWR_FLAG #FLG0101
@@
 	1    0    0    -1
 $EndComp
+$Comp
+L power:VDD #PWR0103
+U 1 1 5DE5EF24
+P 4700 5800
+F 0 "#PWR0103" H 4700 5650 50  0001 C CNN
+F 1 "VDD" H 4717 5973 50  0000 C CNN
+F 2 "" H 4700 5800 50  0001 C CNN
+F 3 "" H 4700 5800 50  0001 C CNN
+	1    4700 5800
+	1    0    0    -1
+$EndComp
+Text Label 5250 5800 0    50   ~ 0
+SWDIO
+Text Label 4400 5900 0    50   ~ 0
+NRESET
+Text Label 5250 5900 0    50   ~ 0
+SWCLK
+$Comp
+L power:GND #PWR0104
+U 1 1 5DE5F92B
+P 4700 6000
+F 0 "#PWR0104" H 4700 5750 50  0001 C CNN
+F 1 "GND" H 4705 5827 50  0000 C CNN
+F 2 "" H 4700 6000 50  0001 C CNN
+F 3 "" H 4700 6000 50  0001 C CNN
+	1    4700 6000
+	1    0    0    -1
+$EndComp
+Wire Wire Line
+	5200 5800 5250 5800
+Wire Wire Line
+	5200 5900 5250 5900
+Wire Wire Line
+	4700 5900 4400 5900
+$Comp
+L sensor_ble:Nrf52810-QCAA U1
+U 1 1 5DC5E292
+P 4050 4450
+F 0 "U1" H 3800 4550 50  0000 L CNN
+F 1 "Nrf52810-QCAA" H 3800 4450 50  0000 L CNN
+F 2 "Package_DFN_QFN:QFN-32-1EP_5x5mm_P0.5mm_EP3.6x3.6mm" H 3600 5200 50  0001 C CNN
+F 3 "" H 3600 5200 50  0001 C CNN
+	1    4050 4450
+	1    0    0    -1
+$EndComp
+Text Label 4400 5500 3    50   ~ 0
+NRESET
+Wire Wire Line
+	4400 5400 4400 5500
+Wire Wire Line
+	5050 4650 5100 4650
+Wire Wire Line
+	5050 4750 5100 4750
+Text Label 5100 4650 0    50   ~ 0
+SWDIO
+Text Label 5100 4750 0    50   ~ 0
+SWCLK
+NoConn ~ 5200 6000
+$Comp
+L Connector_Generic:Conn_02x03_Odd_Even J1
+U 1 1 5DE5D834
+P 4900 5900
+F 0 "J1" H 4900 6150 50  0000 C CNN
+F 1 "TC2030" H 5000 5700 50  0000 C CNN
+F 2 "Connector:Tag-Connect_TC2030-IDC-NL_2x03_P1.27mm_Vertical" H 4900 5900 50  0001 C CNN
+F 3 "~" H 4900 5900 50  0001 C CNN
+	1    4900 5900
+	1    0    0    -1
+$EndComp
+$Comp
+L Device:Antenna_Chip AE1
+U 1 1 5DEA724A
+P 6200 5400
+F 0 "AE1" H 6380 5527 50  0000 L CNN
+F 1 "Antenna_Chip" H 6380 5436 50  0000 L CNN
+F 2 "sensor_ble:2450AT18B100" H 6100 5575 50  0001 C CNN
+F 3 "~" H 6100 5575 50  0001 C CNN
+	1    6200 5400
+	1    0    0    -1
+$EndComp
+$Comp
+L Device:R_Small_US R5
+U 1 1 5DEAEE2E
+P 5900 5500
+F 0 "R5" V 5850 5400 50  0000 C CNN
+F 1 "0" V 5850 5600 50  0000 C CNN
+F 2 "Resistor_SMD:R_0402_1005Metric" H 5900 5500 50  0001 C CNN
+F 3 "~" H 5900 5500 50  0001 C CNN
+	1    5900 5500
+	0    1    1    0
+$EndComp
+$Comp
+L Device:R_Small_US R6
+U 1 1 5DEAF727
+P 5550 5500
+F 0 "R6" V 5500 5450 50  0000 R CNN
+F 1 "NC" V 5500 5650 50  0000 R CNN
+F 2 "Resistor_SMD:R_0402_1005Metric" H 5550 5500 50  0001 C CNN
+F 3 "~" H 5550 5500 50  0001 C CNN
+	1    5550 5500
+	0    1    1    0
+$EndComp
+$Comp
+L Device:R_Small_US R4
+U 1 1 5DEAFF11
+P 5750 5700
+F 0 "R4" H 5682 5654 50  0000 R CNN
+F 1 "NC" H 5682 5745 50  0000 R CNN
+F 2 "Resistor_SMD:R_0402_1005Metric" H 5750 5700 50  0001 C CNN
+F 3 "~" H 5750 5700 50  0001 C CNN
+	1    5750 5700
+	-1   0    0    1
+$EndComp
+$Comp
+L power:GND #PWR0107
+U 1 1 5DEB0B0A
+P 5750 5800
+F 0 "#PWR0107" H 5750 5550 50  0001 C CNN
+F 1 "GND" H 5755 5627 50  0000 C CNN
+F 2 "" H 5750 5800 50  0001 C CNN
+F 3 "" H 5750 5800 50  0001 C CNN
+	1    5750 5800
+	1    0    0    -1
+$EndComp
+Text Label 5150 5500 0    50   ~ 0
+ANT
+Wire Wire Line
+	5050 4550 5100 4550
+Text Label 5100 4550 0    50   ~ 0
+ANT
+Wire Wire Line
+	5650 5500 5750 5500
+Wire Wire Line
+	5750 5600 5750 5500
+Connection ~ 5750 5500
+Wire Wire Line
+	5750 5500 5800 5500
+Wire Wire Line
+	6000 5500 6100 5500
+Wire Wire Line
+	5450 5500 5150 5500
+NoConn ~ 6300 5500
 $EndSCHEMATC

Commit message: Últimas mudanças
Signed-off-by: Rodrigo Peixoto <rodrigopex@ic.ufal.br>
Parts:
- removed H2: MountingHole, MountingHole:MountingHole_2mm, symbol Mechanical:MountingHole
- C14, C3, C5: Part Number (none) -> GCM155L8EH104KE07D
- C7: value N.F. -> NF
- C9: Part Number (none) -> CC0402GRNPO9BN120
- R4, R6: value NC -> NF
Changed lines of the file:
@@
 F 1 "100nF" H 3492 5755 50  0000 L CNN
 F 2 "Capacitor_SMD:C_0402_1005Metric" H 3400 5800 50  0001 C CNN
-F 3 "~" H 3400 5800 50  0001 C CNN
+F 3 "https://br.mouser.com/datasheet/2/281/murata_03122018_GCM_Series-1310150.pdf" H 3400 5800 50  0001 C CNN
+F 4 "GCM155L8EH104KE07D" H 3400 5800 50  0001 C CNN "Part Number"
 	1    3400 5800
 	1    0    0    -1
@@
 F 2 "Capacitor_SMD:C_0402_1005Metric" H 2650 3750 50  0001 C CNN
 F 3 "~" H 2650 3750 50  0001 C CNN
+F 4 "GCM155L8EH104KE07D" H 2650 3750 50  0001 C CNN "Part Number"
 	1    2650 3750
 	1    0    0    -1
@@
 P 4700 2300
 F 0 "C7" H 4792 2346 50  0000 L CNN
-F 1 "N.F." H 4792 2255 50  0000 L CNN
+F 1 "NF" H 4792 2255 50  0000 L CNN
 F 2 "Capacitor_SMD:C_0402_1005Metric" H 4700 2300 50  0001 C CNN
 F 3 "~" H 4700 2300 50  0001 C CNN
@@
 F 1 "12pF" V 6550 3250 50  0000 C CNN
 F 2 "Capacitor_SMD:C_0402_1005Metric" H 6450 3250 50  0001 C CNN
-F 3 "~" H 6450 3250 50  0001 C CNN
+F 3 "https://br.mouser.com/datasheet/2/447/UPY-GP_NP0_16V-to-50V_16-1109089.pdf" H 6450 3250 50  0001 C CNN
+F 4 "CC0402GRNPO9BN120" H 6450 3250 50  0001 C CNN "Part Number"
 	1    6450 3250
 	0    1    1    0
@@
 F 2 "Capacitor_SMD:C_0402_1005Metric" H 10000 2050 50  0001 C CNN
 F 3 "~" H 10000 2050 50  0001 C CNN
+F 4 "GCM155L8EH104KE07D" H 10000 2050 50  0001 C CNN "Part Number"
 	1    10000 2050
 	-1   0    0    -1
@@
 $EndComp
 $Comp
-L Mechanical:MountingHole H2
-U 1 1 5DE39090
-P 4300 7150
-F 0 "H2" H 4400 7196 50  0000 L CNN
-F 1 "MountingHole" H 4400 7105 50  0000 L CNN
-F 2 "MountingHole:MountingHole_2mm" H 4300 7150 50  0001 C CNN
-F 3 "~" H 4300 7150 50  0001 C CNN
-	1    4300 7150
-	1    0    0    -1
-$EndComp
-$Comp
 L power:VDD #PWR0103
 U 1 1 5DE5EF24
@@
 F 1 "Nrf52810-QCAA" H 3800 4450 50  0000 L CNN
 F 2 "Package_DFN_QFN:QFN-32-1EP_5x5mm_P0.5mm_EP3.6x3.6mm" H 3600 5200 50  0001 C CNN
-F 3 "" H 3600 5200 50  0001 C CNN
+F 3 "https://br.mouser.com/datasheet/2/297/nRF52810_PB_v1.1-1146849.pdf" H 3600 5200 50  0001 C CNN
+F 4 "" H 4050 4450 50  0001 C CNN "Part Number"
 	1    4050 4450
 	1    0    0    -1
@@
 F 1 "Antenna_Chip" H 6380 5436 50  0000 L CNN
 F 2 "sensor_ble:2450AT18B100" H 6100 5575 50  0001 C CNN
-F 3 "~" H 6100 5575 50  0001 C CNN
+F 3 "https://br.mouser.com/datasheet/2/611/johanson_2450AT18B100E-1215778.pdf" H 6100 5575 50  0001 C CNN
 	1    6200 5400
 	1    0    0    -1
@@
 P 5550 5500
 F 0 "R6" V 5500 5450 50  0000 R CNN
-F 1 "NC" V 5500 5650 50  0000 R CNN
+F 1 "NF" V 5500 5650 50  0000 R CNN
 F 2 "Resistor_SMD:R_0402_1005Metric" H 5550 5500 50  0001 C CNN
 F 3 "~" H 5550 5500 50  0001 C CNN
@@
 P 5750 5700
 F 0 "R4" H 5682 5654 50  0000 R CNN
-F 1 "NC" H 5682 5745 50  0000 R CNN
+F 1 "NF" H 5682 5745 50  0000 R CNN
 F 2 "Resistor_SMD:R_0402_1005Metric" H 5750 5700 50  0001 C CNN
 F 3 "~" H 5750 5700 50  0001 C CNN
